Commit message: First commit of the popeye arm for PROJ515. Works (with cartesian control of the EE), but the wrist is upside-down and sometimes forearm_roll oscillates

File: xacro/gummi_description_ee.urdf.xacro (robot description, xacro)
@@ -136,76 +136,3 @@
       <limit effort="0" lower="-1.5" upper="1.68" velocity="1.0"/>
   </joint>
-  <!-- gripper_Link -->
-  <link
-    name="gripper_Link">
-    <inertial>
-      <origin
-        xyz="-0.0233988267408998 -0.0183769778598925 -0.00217479089040148"
-        rpy="0 0 0" />
-      <mass
-        value="0.0573612129510164" />
-      <inertia
-        ixx="1.07017574054092E-05"
-        ixy="1.20541476778111E-07"
-        ixz="-2.08068523476524E-06"
-        iyy="6.40757036666839E-05"
-        iyz="3.89770387703761E-08"
-        izz="6.62562645856636E-05" />
-    </inertial>
-    <visual>
-      <origin
-        xyz="0.05 0 0"
-        rpy="0 0 0" />
-      <geometry>
-        <box size=".07 .008 .06" />
-      </geometry>
-      <material
-        name="">
-        <color
-          rgba="0.79216 0.81961 0.93333 1" />
-      </material>
-    </visual>
-    <collision>
-      <origin
-        xyz="0.05 0 0"
-        rpy="0 0 0" />
-      <geometry>
-        <box size=".07 .008 .06" />
-      </geometry>
-    </collision>
-  </link>
-  <!-- gripper -->
-  <joint
-    name="gripper"
-    type="revolute">
-    <origin
-      xyz="0.14 0 0"
-      rpy="1.5708 1.0472 3.1416" />
-    <parent
-      link="wrist" />
-    <child
-      link="gripper_Link" />
-    <axis
-      xyz="0 0 1" />
-    <!-- <limit
-      lower="-1.5708"
-      upper="1.5708"
-      effort="0"
-      velocity="0" /> -->
-    <limit effort="0" lower="-2.0" upper="0.37" velocity="1.0"/>
-  </joint>
-  <link name="tool">
-  </link>
-  <joint name="coupling_tool" type="fixed">
-    <origin rpy="0 0 0" xyz="0.175 -0.02 0.13"/>
-    <parent link="wrist"/>
-    <child link="tool"/>
-    <axis xyz="0 1 0"/>
-    <!-- <limit
-    lower="-1.5708"
-    upper="1.5708"
-    effort="0"
-    velocity="0" /> -->
-    <limit effort="0" lower="-0.30" upper="0.17" velocity="1.0"/>
-  </joint>
 </robot>

File: xacro/gummi_ee.srdf.xacro (robot description, xacro)
@@ -5,12 +5,10 @@
     <joint name="forearm_roll" />
     <joint name="wrist_pitch" />
-    <joint name="coupling_tool"/>
 </xacro:macro>
-<xacro:macro name="group_right_gripper_ee">
+<!--xacro:macro name="group_right_gripper_ee">
   <group name="right_gripper">
       <link name="wrist" />
-      <link name="gripper_Link" />
   </group>
-</xacro:macro>
+</xacro:macro-->
 <xacro:macro name="group_state_right_arm_ee">
   <joint name="elbow" value="0" />
@@ -18,17 +16,16 @@
   <joint name="wrist_pitch" value="0" />
 </xacro:macro>
+<!--
 <xacro:macro name="end_effector_ee">
-  <!--END EFFECTOR: Purpose: Represent information about an end effector.-->
 <end_effector group="right_arm" name="right_eef" parent_link="tool"/>
-</xacro:macro>
+</xacro:macro-->
 <xacro:macro name="disable_collisions_ee">
   <!-- <disable_collisions link1="right_hand" link2="wrist" reason="Never" />
   <disable_collisions link1="right_hand" link2="gripper_Link" reason="Never" /> -->
-  <disable_collisions link1="gripper_Link" link2="lowerarm" reason="Never" />
-  <disable_collisions link1="gripper_Link" link2="lowerarm_preroll_d" reason="Never" />
-  <disable_collisions link1="gripper_Link" link2="wrist" reason="Adjacent" />
   <disable_collisions link1="lowerarm" link2="lowerarm_preroll_d" reason="Adjacent" />
   <disable_collisions link1="lowerarm" link2="wrist" reason="Adjacent" />
   <disable_collisions link1="lowerarm_preroll_d" link2="wrist" reason="Never" />
+  <disable_collisions link1="lowerarm_preroll_d" link2="lowerarm_preroll_u" reason="Never" />
+  <disable_collisions link1="lowerarm_preroll_u" link2="wrist" reason="Never" />
 </xacro:macro>
 </robot>
